File: KosmosV4System/hardware/CartesElectroniques/RPi_PCB_3-sansfioriture_alternative/RPi_PCB_KOSMOS_4.0_uptodate - Copie/RPi_PCB_KOSMOS_4.0_v2.kicad_pcb (KiCad board)
At the start: 2 copper layers, 65.7 x 58.7 mm, 13 parts, among them IC1 Module_GPS, J1 Raspberry_Pi_2_3, J2 Arduino_Motor, J4 Capteur_Temp, J9 Capteur_Magneto, J9 Capteur_TP

Commit message: kh
Parts:
- added ?: , , F.Cu at (163.2, 75.4)
- added ?: , , F.Cu at (169.9, 64.0)
Other:
- board size 65.7 x 58.7 mm -> 65.7 x 58.8 mm
Changed lines of the file:
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@@
 		)
 	)
+	(footprint ""
+		(layer "F.Cu")
+		(at 163.2 75.4)
+		(property "Reference" ""
+			(at 0 0 0)
+			(layer "F.SilkS")
+			(effects
+				(font
+					(size 1.27 1.27)
+					(thickness 0.15)
+				)
+			)
+		)
+		(property "Value" ""
+			(at 0 0 0)
+			(layer "F.Fab")
+			(effects
+				(font
+					(size 1.27 1.27)
+					(thickness 0.15)
+				)
+			)
+		)
+		(property "Footprint" ""
+			(at 0 0 0)
+			(layer "F.Fab")
+			(hide yes)
+			(effects
+				(font
+					(size 1.27 1.27)
+					(thickness 0.15)
+				)
+			)
+		)
+		(property "Datasheet" ""
+			(at 0 0 0)
+			(layer "F.Fab")
+			(hide yes)
+			(effects
+				(font
+					(size 1.27 1.27)
+					(thickness 0.15)
+				)
+			)
+		)
+		(property "Description" ""
+			(at 0 0 0)
+			(layer "F.Fab")
+			(hide yes)
+			(effects
+				(font
+					(size 1.27 1.27)
+					(thickness 0.15)
+				)
+			)
+		)
+		(pad "2" thru_hole roundrect
+			(at 0 0 270)
+			(size 2.2 2.2)
+			(drill 1)
+			(layers "*.Cu" "*.Mask")
+			(remove_unused_layers no)
+			(roundrect_rratio 0.1136363636)
+			(net 9 "GND")
+			(pinfunction "-")
+			(pintype "passive")
+		)
+	)
 	(footprint "Library_komsos:MountingHole_2.2mm_M2"
 		(layer "F.Cu")
@@
 		)
 	)
+	(footprint ""
+		(layer "F.Cu")
+		(at 169.9 64)
+		(property "Reference" ""
+			(at 0 0 0)
+			(layer "F.SilkS")
+			(effects
+				(font
+					(size 1.27 1.27)
+					(thickness 0.15)
+				)
+			)
+		)
+		(property "Value" ""
+			(at 0 0 0)
+			(layer "F.Fab")
+			(effects
+				(font
+					(size 1.27 1.27)
+					(thickness 0.15)
+				)
+			)
+		)
+		(property "Footprint" ""
+			(at 0 0 0)
+			(layer "F.Fab")
+			(hide yes)
+			(effects
+				(font
+					(size 1.27 1.27)
+					(thickness 0.15)
+				)
+			)
+		)
+		(property "Datasheet" ""
+			(at 0 0 0)
+			(layer "F.Fab")
+			(hide yes)
+			(effects
+				(font
+					(size 1.27 1.27)
+					(thickness 0.15)
+				)
+			)
+		)
+		(property "Description" ""
+			(at 0 0 0)
+			(layer "F.Fab")
+			(hide yes)
+			(effects
+				(font
+					(size 1.27 1.27)
+					(thickness 0.15)
+				)
+			)
+		)
+		(pad "2" thru_hole roundrect
+			(at 0 0 270)
+			(size 2.2 2.2)
+			(drill 1)
+			(layers "*.Cu" "*.Mask")
+			(remove_unused_layers no)
+			(roundrect_rratio 0.1136363636)
+			(net 9 "GND")
+			(pinfunction "-")
+			(pintype "passive")
+		)
+	)
 	(footprint "Library_komsos:R_Axial_DIN0207_L6.3mm_D2.5mm_P10.16mm_Horizontal_v2.2mm"
 		(layer "F.Cu")
@@
 	)
 	(gr_line
-		(start 201.7 105.6)
+		(start 201.7 105.8)
 		(end 201.7 73.5)
 		(stroke
@@
 	(gr_line
 		(start 145.6 105.7)
-		(end 201.7 105.6)
+		(end 201.8 105.7)
 		(stroke
 			(width 0.05)
@@
 		(layer "B.Cu")
 		(net 9)
+	)
+	(segment
+		(start 163.26 75.34)
+		(end 163.2 75.4)
+		(width 0.8)
+		(layer "B.Cu")
+		(net 9)

Commit message: fghjfghj
Parts:
- removed the ? at (153.7, 76.6)
- moved J9 3.61 mm to (188.4, 84.6)
- moved J9 3.61 mm to (167.7, 84.7)
- moved J4 3.60 mm to (192.9, 92.1)
- moved ? 3.47 mm to (164.8, 78.5)
Routing:
- net RX: track 3.94 -> 0.06 mm
- net +3.3V: track 71.2 -> 75.0 mm
- net SCL: track 86.3 -> 89.6 mm
- net SDA: track 82.2 -> 85.3 mm
Changed lines of the file:
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@@
 		)
 	)
-	(footprint ""
-		(layer "F.Cu")
-		(at 153.7 76.6)
-		(property "Reference" ""
-			(at 0 0 0)
-			(layer "F.SilkS")
-			(effects
-				(font
-					(size 1.27 1.27)
-					(thickness 0.15)
-				)
-			)
-		)
-		(property "Value" ""
-			(at 0 0 0)
-			(layer "F.Fab")
-			(effects
-				(font
-					(size 1.27 1.27)
-					(thickness 0.15)
-				)
-			)
-		)
-		(property "Footprint" ""
-			(at 0 0 0)
-			(layer "F.Fab")
-			(hide yes)
-			(effects
-				(font
-					(size 1.27 1.27)
-					(thickness 0.15)
-				)
-			)
-		)
-		(property "Datasheet" ""
-			(at 0 0 0)
-			(layer "F.Fab")
-			(hide yes)
-			(effects
-				(font
-					(size 1.27 1.27)
-					(thickness 0.15)
-				)
-			)
-		)
-		(property "Description" ""
-			(at 0 0 0)
-			(layer "F.Fab")
-			(hide yes)
-			(effects
-				(font
-					(size 1.27 1.27)
-					(thickness 0.15)
-				)
-			)
-		)
-		(pad "2" thru_hole circle
-			(at 0 0 270)
-			(size 2.2 2.2)
-			(drill 1)
-			(layers "*.Cu" "*.Mask")
-			(remove_unused_layers no)
-			(net 8 "RX")
-			(pinfunction "-")
-			(pintype "passive")
-		)
-	)
 	(footprint "Library_komsos:GPS_BDS_BeiDou_Dual_Module_v2.2mm"
 		(layer "F.Cu")
@@
 	(footprint ""
 		(layer "F.Cu")
-		(at 163.2 75.4)
+		(at 164.84 78.46)
 		(property "Reference" ""
 			(at 0 0 0)
@@
 	(footprint "Library_komsos:JST_EH_S4B-EH_1x04_P2.50mm_Horizontal_kosmos"
 		(layer "B.Cu")
-		(at 188.1 81 -90)
+		(at 188.4 84.6 -90)
 		(descr "JST EH series connector, S4B-EH (http://www.jst-mfg.com/product/pdf/eng/eEH.pdf), generated with kicad-footprint-generator")
 		(tags "connector JST EH horizontal")
@@
 	(footprint "Library_komsos:JST_EH_S4B-EH_1x04_P2.50mm_Horizontal_kosmos"
 		(layer "B.Cu")
-		(at 192.9 88.5 90)
+		(at 192.9 92.1 90)
 		(descr "JST EH series connector, S4B-EH (http://www.jst-mfg.com/product/pdf/eng/eEH.pdf), generated with kicad-footprint-generator")
 		(tags "connector JST EH horizontal")
@@
 	(footprint "Library_komsos:JST_EH_S4B-EH_1x04_P2.50mm_Horizontal_kosmos"
 		(layer "B.Cu")
-		(at 167.9 81.1 -90)
+		(at 167.7 84.7 -90)
 		(descr "JST EH series connector, S4B-EH (http://www.jst-mfg.com/product/pdf/eng/eEH.pdf), generated with kicad-footprint-generator")
 		(tags "connector JST EH horizontal")
@@
 	)
 	(segment
-		(start 167.9 88.6)
-		(end 158.84 88.6)
+		(start 188.3 92.2)
+		(end 188.4 92.1)
+		(width 0.8)
+		(layer "B.Cu")
+		(net 6)
+	)
+	(segment
+		(start 167.8 92.1)
+		(end 167.7 92.2)
 		(width 0.8)
 		(layer "B.Cu")
@@
 	)
 	(segment
-		(start 188 88.6)
-		(end 188.1 88.5)
+		(start 158.84 92.16)
+		(end 158.8 92.2)
 		(width 0.8)
 		(layer "B.Cu")
@@
 	)
 	(segment
-		(start 188.1 88.5)
-		(end 192.9 88.5)
+		(start 192.9 92.1)
+		(end 167.8 92.1)
 		(width 0.8)
 		(layer "B.Cu")
@@
 	)
 	(segment
-		(start 158.84 88.6)
-		(end 158.84 72.745)
+		(start 158.8 92.2)
+		(end 167.7 92.2)
 		(width 0.8)
 		(layer "B.Cu")
@@
 	)
 	(segment
-		(start 167.9 88.6)
-		(end 188 88.6)
+		(start 158.84 72.745)
+		(end 158.84 92.16)
 		(width 0.8)
 		(layer "B.Cu")
@@
 	)
 	(segment
-		(start 153.76 72.745)
-		(end 153.76 76.54)
-		(width 0.8)
-		(layer "B.Cu")
-		(net 8)
-	)
-	(segment
 		(start 153.8 72.705)
 		(end 153.76 72.745)
@@
 	)
 	(segment
-		(start 153.76 76.54)
-		(end 153.7 76.6)
-		(width 0.8)
-		(layer "B.Cu")
-		(net 8)
-	)
-	(segment
-		(start 187.7 85.9)
-		(end 187.8 86)
+		(start 188 89.5)
+		(end 188.1 89.6)
 		(width 0.8)
 		(layer "B.Cu")
@@
 	)
 	(segment
-		(start 168 86)
-		(end 167.9 86.1)
-		(width 1.5)
-		(layer "B.Cu")
-		(net 9)
-	)
-	(segment
-		(start 163.26 75.34)
-		(end 163.2 75.4)
+		(start 164.9 78.4)
+		(end 164.84 78.46)
 		(width 0.8)
 		(layer "B.Cu")
@@
 	)
 	(segment
-		(start 192.7 81.2)
-		(end 192.9 81)
-		(width 0.8)
-		(layer "B.Cu")
-		(net 21)
-	)
-	(segment
-		(start 192.9 74.5)
-		(end 192.9 81)
-		(width 0.8)
-		(layer "B.Cu")
-		(net 21)
-	)
-	(segment
-		(start 192.9 81)
-		(end 188.1 81)
-		(width 0.8)
-		(layer "B.Cu")
-		(net 21)
-	)
-	(segment
-		(start 167.9 81.1)
-		(end 188 81.1)
+		(start 192.9 84.6)
+		(end 167.8 84.6)
 		(width 0.8)
 		(layer "B.Cu")
@@
 	)
 	(segment
-		(start 192.8 80.9)
-		(end 192.9 81)
+		(start 192.9 74.5)
+		(end 192.9 84.6)
 		(width 0.8)
 		(layer "B.Cu")
@@
 	)
 	(segment
-		(start 188 81.1)
-		(end 188.1 81)
+		(start 167.8 84.6)
+		(end 167.7 84.7)
 		(width 0.8)
 		(layer "B.Cu")
@@
 	)
 	(segment
-		(start 192.6 80.7)
-		(end 192.9 81)
+		(start 188.3 84.7)
+		(end 188.4 84.6)
 		(width 0.8)
 		(layer "B.Cu")
@@
 	)
 	(segment
-		(start 167.9 83.6)
-		(end 188 83.6)
-		(width 0.8)
-		(layer "B.Cu")
-		(net 26)
-	)
-	(segment
 		(start 159.48 54.27)
 		(end 159.48 63.08)
@@
 	)
 	(segment
-		(start 187.7 83.4)
-		(end 187.8 83.5)
+		(start 188 87)
+		(end 188.1 87.1)
 		(width 0.8)
 		(layer "B.Cu")
@@
 	)
 	(segment
-		(start 159.48 63.08)
-		(end 168.4 72)
+		(start 192.9 87.1)
+		(end 167.8 87.1)
 		(width 0.8)
 		(layer "B.Cu")
@@
 	)
 	(segment
-		(start 188 83.6)
-		(end 188.1 83.5)
+		(start 167.8 87.1)
+		(end 167.7 87.2)
 		(width 0.8)
 		(layer "B.Cu")
@@
 	)
 	(segment
-		(start 192.9 83.5)
-		(end 188.1 83.5)
+		(start 159.48 63.08)
+		(end 168.4 72)
 		(width 0.8)
 		(layer "B.Cu")
@@
 	)
 	(segment
-		(start 195.4 81)
-		(end 192.9 83.5)
+		(start 188.3 87.2)
+		(end 188.4 87.1)
 		(width 0.8)
 		(layer "B.Cu")
@@
 	)
 	(segment
-		(start 159.48 54.27)
-		(end 159.9 54.69)
+		(start 194.6 85.4)
+		(end 192.9 87.1)
 		(width 0.8)
 		(layer "B.Cu")
@@
 	)
 	(segment
-		(start 195.4 74.5)
-		(end 195.4 81)
+		(start 159.48 54.27)
+		(end 159.9 54.69)
 		(width 0.8)
 		(layer "B.Cu")
@@
 	(segment
 		(start 192.9 72)
-		(end 195.4 74.5)
+		(end 194.6 73.7)
+		(width 0.8)
+		(layer "B.Cu")
+		(net 26)
+	)
+	(segment
+		(start 194.6 73.7)
+		(end 194.6 85.4)
 		(width 0.8)
 		(layer "B.Cu")
