File: KosmosV4System/hardware/CartesElectroniques/RPi_PCB_2/RPi_PCB_KOSMOS_4.0_uptodate - Copie/RPi_PCB_KOSMOS_4.0_v2.kicad_pcb (KiCad board)
At the start: 2 copper layers, 85.4 x 58.5 mm, 22 parts, among them IC1 Module_GPS, J1 Raspberry_Pi_2_3, J2 Arduino_Motor, J4 Capteur_Temp, J5 Conn_01x01_Socket_Solder_Pad, J6 Conn_01x01_Socket_Solder_Pad, J7 Alim_Principale, J9 Capteur_Lux, J9 Capteur_Magneto, SW1 SW_REC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

Commit message: dfh
Parts:
- added REF**: MountingHole_2.2mm_M2, Library_komsos:MountingHole_2.2mm_M2, F.Cu at (211.1, 102.0)
Changed lines of the file:
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@@
+		)
+	)
+	(footprint "Library_komsos:MountingHole_2.2mm_M2"
+		(layer "F.Cu")
+		(at 211.1 102)
+		(descr "Mounting Hole 2.2mm, no annular, M2")
+		(tags "mounting hole 2.2mm no annular m2")
+		(property "Reference" "REF**"
+			(at 0 -3.2 0)
+			(layer "F.SilkS")
+			(effects
+				(font
+					(size 1 1)
+					(thickness 0.15)
+				)
+			)
+		)
+		(property "Value" "MountingHole_2.2mm_M2"
+			(at 0 3.2 0)
+			(layer "F.Fab")
+			(effects
+				(font
+					(size 1 1)
+					(thickness 0.15)
+				)
+			)
+		)
+		(property "Footprint" "Library_komsos:MountingHole_2.2mm_M2"
+			(at 0 0 0)
+			(unlocked yes)
+			(layer "F.Fab")
+			(hide yes)
+			(effects
+				(font
+					(size 1.27 1.27)
+					(thickness 0.15)
+				)
+			)
+		)
+		(property "Datasheet" ""
+			(at 0 0 0)
+			(unlocked yes)
+			(layer "F.Fab")
+			(hide yes)
+			(effects
+				(font
+					(size 1.27 1.27)
+					(thickness 0.15)
+				)
+			)
+		)
+		(property "Description" ""
+			(at 0 0 0)
+			(unlocked yes)
+			(layer "F.Fab")
+			(hide yes)
+			(effects
+				(font
+					(size 1.27 1.27)
+					(thickness 0.15)
+				)
+			)
+		)
+		(attr exclude_from_pos_files exclude_from_bom)
+		(fp_circle
+			(center 0 0)
+			(end 2.2 0)
+			(stroke
+				(width 0.15)
+				(type solid)
+			)
+			(fill none)
+			(layer "Cmts.User")
+		)
+		(fp_circle
+			(center 0 0)
+			(end 2.45 0)
+			(stroke
+				(width 0.05)
+				(type solid)
+			)
+			(fill none)
+			(layer "F.CrtYd")
+		)
+		(fp_text user "${REFERENCE}"
+			(at 0 0 0)
+			(layer "F.Fab")
+			(effects
+				(font
+					(size 1 1)
+					(thickness 0.15)
+				)
+			)
+		)
+		(pad "" np_thru_hole circle
+			(at 0 0)
+			(size 2.2 2.2)
+			(drill 2.2)
+			(layers "F&B.Cu" "*.Mask")
+			(clearance 0.5)
 		)
 	)
