File: KosmosV4System/hardware/CartesElectroniques/RPi_PCB_v4.2/RPi_PCB_KOSMOS_4.0_uptodate - Copie/RPi_PCB_KOSMOS_4.0_v2.kicad_pcb (KiCad board)
At the start: 2 copper layers, 66.2 x 58.5 mm, 21 parts, among them IC1 Module_GPS, J1 Raspberry_Pi_2_3, J2 Arduino_Motor, J3 ILS 1, J4 Capteur_Temp, J5 Conn_01x01_Socket_Solder_Pad, J6 Conn_01x01_Socket_Solder_Pad, J7 Alim_Principale, J9 Capteur_Lux

Commit message: hfgdh
Parts:
- moved ? 5.28 mm to (153.4, 83.5)
- moved J7 3.82 mm to (205.9, 68.3)
- moved J6 3.32 mm to (197.8, 68.3)
- moved ? 2.52 mm to (163.2, 83.5)
- moved J5 0.81 mm to (151.9, 60.3)
- moved J9 0.45 mm to (165.9, 89.5)
- moved REF** 0.29 mm to (170.9, 96.8)
Routing:
- net GND: track 4.32 -> 0.00 mm, vias 1 -> 0
- net +3.3V: track 79.2 -> 83.0 mm
- net SCL: track 84.3 -> 81.2 mm
- net GPIO27: track 23.1 -> 22.1 mm
- net GPIO17: track 13.3 -> 12.5 mm
- net GPIO5: track 16.6 -> 15.9 mm
- net SDA: track 78.2 -> 77.6 mm
Other:
- board size 66.2 x 58.5 mm -> 66.3 x 58.5 mm
